Commit message: chore: set up rviz bringup

File: ros2_ws/src/robocup_description/urdf/robot.urdf.xacro (robot description, xacro)
@@ -1,4 +1,10 @@
 <?xml version="1.0"?>
 <robot xmlns:xacro="http://www.ros.org/wiki/xacro" name="robocup_robot">
+  <link name="base_link_footprint"/>
+  <joint name="base_joint" type="fixed">
+    <parent link="base_link_footprint"/>
+    <child link="base_link"/>
+    <origin xyz="0 0 0" rpy="0 0 0"/>
+  </joint>
   <link name="base_link">
     <visual>

Commit message: feat: add xacro wheels and joint state publisher

File: ros2_ws/src/robocup_description/urdf/robot.urdf.xacro (robot description, xacro)
@@ -1,29 +1,69 @@
 <?xml version="1.0"?>
 <robot xmlns:xacro="http://www.ros.org/wiki/xacro" name="robocup_robot">
-  <link name="base_link_footprint"/>
+  <link name="base_footprint"/>
   <joint name="base_joint" type="fixed">
-    <parent link="base_link_footprint"/>
+    <parent link="base_footprint"/>
     <child link="base_link"/>
-    <origin xyz="0 0 0" rpy="0 0 0"/>
+    <origin xyz="0 0 0.10" rpy="0 0 0"/>
   </joint>
   <link name="base_link">
     <visual>
       <geometry>
-        <box size="0.5 0.4 0.15"/>
+        <box size="0.6 0.48 0.2"/>
       </geometry>
     </visual>
     <collision>
       <geometry>
-        <box size="0.5 0.4 0.15"/>
+        <box size="0.6 0.48 0.2"/>
       </geometry>
     </collision>
     <inertial>
-      <mass value="10.0"/>
+      <mass value="13.96"/>
       <origin xyz="0 0 0"/>
       <inertia
-        ixx="0.15" ixy="0" ixz="0"
-        iyy="0.2" iyz="0"
-        izz="0.25"/>
+        ixx="0.315" ixy="0" ixz="0"
+        iyy="0.466" iyz="0"
+        izz="0.687"/>
     </inertial>
   </link>
+  <xacro:macro name="wheel" params="name parent origin">
+    <link name="${name}">
+      <visual>
+        <origin xyz="0 0 0" rpy="1.5708 0 0"/>
+        <geometry>
+          <cylinder radius="0.075" length="0.05"/>
+        </geometry>
+        <material name="white">
+          <color rgba="1 1 1 1"/>
+        </material>
+      </visual>
+      <collision>
+        <origin xyz="0 0 0" rpy="1.5708 0 0"/>
+        <geometry>
+          <cylinder radius="0.075" length="0.05"/>
+        </geometry>
+      </collision>
+      <inertial>
+        <mass value="0.975"/>
+        <origin xyz="0 0 0"/>
+       <inertia
+          ixx="0.001574"
+          ixy="0"
+          ixz="0"
+          iyy="0.002742"
+          iyz="0"
+          izz="0.001574"/>
+      </inertial>
+    </link>
+    <joint name="${name}_joint" type="continuous">
+      <parent link="${parent}"/>
+      <child link="${name}"/>
+      <origin xyz="${origin}" rpy="0 0 0"/>
+      <axis xyz="0 1 0"/>
+    </joint>
+  </xacro:macro>
+  <xacro:wheel name="rear_left_wheel" parent="base_link" origin="-0.275 0.265 -0.030"/>
+  <xacro:wheel name="rear_right_wheel" parent="base_link" origin="-0.275 -0.265 -0.030"/>
+  <xacro:wheel name="front_left_wheel" parent="base_link" origin="0.275 0.265 -0.03"/>
+  <xacro:wheel name="front_right_wheel" parent="base_link" origin="0.275 -0.265 -0.03"/>
 </robot>

Commit message: feat: add gazebo-hardware  custom implementation

File: ros2_ws/src/robocup_description/urdf/robot.urdf.xacro (robot description, xacro)
@@ -67,3 +67,21 @@
   <xacro:wheel name="front_left_wheel" parent="base_link" origin="0.275 0.265 -0.03"/>
   <xacro:wheel name="front_right_wheel" parent="base_link" origin="0.275 -0.265 -0.03"/>
+  <ros2_control name="GazeboSystem" type="system">
+    <hardware>
+      <plugin>robocup_hardware/GazeboHardware</plugin>
+    </hardware>
+      <joint name="front_left_wheel_joint">
+        <command_interface name="velocity"/>
+        <state_interface name="position"/>
+        <state_interface name="velocity"/>
+      </joint>
+  </ros2_control>
+  <xacro:arg name="controllers_file" default=""/>
+  <gazebo>
+    <plugin
+      filename="libgz_ros2_control-system.so"
+      name="gz_ros2_control::GazeboSimROS2ControlPlugin">
+      <parameters>$(arg controllers_file)</parameters>
+    </plugin>
+</gazebo>
 </robot>

Commit message: feat: add support for 4 wheels

File: ros2_ws/src/robocup_description/urdf/robot.urdf.xacro (robot description, xacro)
@@ -76,4 +76,19 @@
         <state_interface name="velocity"/>
       </joint>
+      <joint name="front_right_wheel_joint">
+        <command_interface name="velocity"/>
+        <state_interface name="position"/>
+        <state_interface name="velocity"/>
+      </joint>
+      <joint name="rear_left_wheel_joint">
+        <command_interface name="velocity"/>
+        <state_interface name="position"/>
+        <state_interface name="velocity"/>
+      </joint>
+      <joint name="rear_right_wheel_joint">
+        <command_interface name="velocity"/>
+        <state_interface name="position"/>
+        <state_interface name="velocity"/>
+      </joint>
   </ros2_control>
   <xacro:arg name="controllers_file" default=""/>

Commit message: feat: add mecanum support

File: ros2_ws/src/robocup_description/urdf/robot.urdf.xacro (robot description, xacro)
@@ -1,9 +1,9 @@
 <?xml version="1.0"?>
-<robot xmlns:xacro="http://www.ros.org/wiki/xacro" name="robocup_robot">
+<robot xmlns:xacro="http://www.ros.org/wiki/xacro" xmlns:ignition="http://gazebosim.org/schema" name="robocup_robot">
   <link name="base_footprint"/>
   <joint name="base_joint" type="fixed">
     <parent link="base_footprint"/>
     <child link="base_link"/>
-    <origin xyz="0 0 0.10" rpy="0 0 0"/>
+    <origin xyz="0 0 0.1" rpy="0 0 0"/>
   </joint>
   <link name="base_link">
@@ -41,5 +41,5 @@
         <origin xyz="0 0 0" rpy="1.5708 0 0"/>
         <geometry>
-          <cylinder radius="0.075" length="0.05"/>
+          <sphere radius="0.075" />
         </geometry>
       </collision>
@@ -60,11 +60,66 @@
       <child link="${name}"/>
       <origin xyz="${origin}" rpy="0 0 0"/>
+      <dynamics damping="0.2"/>
       <axis xyz="0 1 0"/>
     </joint>
   </xacro:macro>
-  <xacro:wheel name="rear_left_wheel" parent="base_link" origin="-0.275 0.265 -0.030"/>
-  <xacro:wheel name="rear_right_wheel" parent="base_link" origin="-0.275 -0.265 -0.030"/>
-  <xacro:wheel name="front_left_wheel" parent="base_link" origin="0.275 0.265 -0.03"/>
-  <xacro:wheel name="front_right_wheel" parent="base_link" origin="0.275 -0.265 -0.03"/>
+  <xacro:wheel name="rear_left_wheel" parent="base_link" origin="-0.275 0.265 -0.070"/>
+  <xacro:wheel name="rear_right_wheel" parent="base_link" origin="-0.275 -0.265 -0.070"/>
+  <xacro:wheel name="front_left_wheel" parent="base_link" origin="0.275 0.265 -0.07"/>
+  <xacro:wheel name="front_right_wheel" parent="base_link" origin="0.275 -0.265 -0.07"/>
+  <!-- To emulate Mecanum wheels in Gazebo with spherical collisions it
+  requires a custom friction model so the vehicle can strafe left to right -->
+  <gazebo reference='front_left_wheel'>
+    <collision>
+      <surface>
+        <friction>
+          <ode>
+            <mu>0</mu>
+            <mu2>0</mu2>
+            <fdir1 ignition:expressed_in="base_link">1.0 1.0 0.0</fdir1>
+          </ode>
+        </friction>
+      </surface>
+    </collision>
+  </gazebo>
+  <gazebo reference='front_right_wheel'>
+    <collision>
+      <surface>
+        <friction>
+          <ode>
+            <mu>0</mu>
+            <mu2>0</mu2>
+            <fdir1 ignition:expressed_in="base_link">1.0 -1.0 0.0</fdir1>
+          </ode>
+        </friction>
+      </surface>
+    </collision>
+  </gazebo>
+  <gazebo reference='rear_left_wheel'>
+    <collision>
+      <surface>
+        <friction>
+          <ode>
+            <mu>0</mu>
+            <mu2>0</mu2>
+            <fdir1 ignition:expressed_in="base_link">1.0 -1.0 0.0</fdir1>
+          </ode>
+        </friction>
+      </surface>
+    </collision>
+  </gazebo>
+  <gazebo reference='rear_right_wheel'>
+    <collision>
+      <surface>
+        <friction>
+          <ode>
+            <mu>0</mu>
+            <mu2>0</mu2>
+            <fdir1 ignition:expressed_in="base_link">1.0 1.0 0.0</fdir1>
+          </ode>
+        </friction>
+      </surface>
+    </collision>
+  </gazebo>
   <ros2_control name="GazeboSystem" type="system">
     <hardware>
@@ -98,4 +153,5 @@
       name="gz_ros2_control::GazeboSimROS2ControlPlugin">
       <parameters>$(arg controllers_file)</parameters>
+      <ros> <remapping>/mecanum_drive_controller/reference:=/cmd_vel</remapping> </ros>
     </plugin>
 </gazebo>

Commit message: feat: add lidar support and mapping with slam

File: ros2_ws/src/robocup_description/urdf/robot.urdf.xacro (robot description, xacro)
@@ -68,4 +68,64 @@
   <xacro:wheel name="front_left_wheel" parent="base_link" origin="0.275 0.265 -0.07"/>
   <xacro:wheel name="front_right_wheel" parent="base_link" origin="0.275 -0.265 -0.07"/>
+  <joint name="sensor_joint" type="fixed">
+    <parent link="base_link"/>
+    <child link="sensor_link"/>
+    <origin xyz="0.3 0 0.125" rpy="0.0 0.0 0.0"/>
+  </joint>
+  <link name="sensor_link">
+    <visual >
+      <origin xyz="0.0 0.0 0.0" rpy="0.0 0.0 0.0"/>
+      <geometry>
+        <box size="0.1 0.005 0.005"/>
+      </geometry>
+      <material name="white">
+        <color rgba="1.0 0.0 0.0 1.0"/>
+      </material>
+    </visual>
+    <collision>
+      <origin xyz="0.0 0.0 0.0" rpy="0.0 0.0 0.0"/>
+      <geometry>
+        <box size="0.1 0.005 0.005"/>
+      </geometry>
+    </collision>
+    <inertial>
+      <mass value="0.1"/> <!-- Obligatorio para que Gazebo procese el sensor -->
+      <origin xyz="0 0 0" rpy="0 0 0"/>
+      <inertia
+        ixx="0.00004" ixy="0" ixz="0"
+        iyy="0.00004" iyz="0"
+        izz="0.00004"/>
+    </inertial>
+  </link>
+  <gazebo reference='sensor_link'>
+    <sensor name='gpu_lidar' type='gpu_lidar'>
+          <pose>0 0 0 0 0 0</pose>
+          <topic>scan</topic>
+           <ignition_frame_id>sensor_link</ignition_frame_id>
+          <update_rate>10</update_rate>
+          <lidar>
+            <scan>
+              <horizontal>
+                <samples>640</samples>
+                <resolution>1</resolution>
+                <min_angle>-1.396263</min_angle>
+                <max_angle>1.396263</max_angle>
+              </horizontal>
+              <vertical>
+                <samples>1</samples>
+                <resolution>1</resolution>
+                <min_angle>0.0</min_angle>
+                <max_angle>0.0</max_angle>
+              </vertical>
+            </scan>
+            <range>
+              <min>0.08</min>
+              <max>10.0</max>
+              <resolution>0.01</resolution>
+            </range>
+          </lidar>
+          <visualize>true</visualize>
+        </sensor>
+      </gazebo>
   <!-- To emulate Mecanum wheels in Gazebo with spherical collisions it
   requires a custom friction model so the vehicle can strafe left to right -->
@@ -153,5 +213,9 @@
       name="gz_ros2_control::GazeboSimROS2ControlPlugin">
       <parameters>$(arg controllers_file)</parameters>
-      <ros> <remapping>/mecanum_drive_controller/reference:=/cmd_vel</remapping> </ros>
+      <ros>
+        <remapping>/mecanum_drive_controller/reference:=/cmd_vel</remapping>
+        <remapping>/mecanum_drive_controller/odometry:=/odom</remapping>
+        <remapping>/mecanum_drive_controller/tf_odometry:=/tf</remapping>
+      </ros>
     </plugin>
 </gazebo>

Commit message: feat: enhance inco world

File: ros2_ws/src/robocup_description/urdf/robot.urdf.xacro (robot description, xacro)
@@ -12,4 +12,5 @@
         <box size="0.6 0.48 0.2"/>
       </geometry>
+      <material name="body_teal"><color rgba="0.04 0.42 0.48 1"/></material>
     </visual>
     <collision>
@@ -34,6 +35,6 @@
           <cylinder radius="0.075" length="0.05"/>
         </geometry>
-        <material name="white">
-          <color rgba="1 1 1 1"/>
+        <material name="wheel_rubber">
+          <color rgba="0.055 0.065 0.075 1"/>
         </material>
       </visual>
@@ -80,5 +81,5 @@
       </geometry>
       <material name="white">
-        <color rgba="1.0 0.0 0.0 1.0"/>
+        <color rgba="0.96 0.64 0.12 1.0"/>
       </material>
     </visual>
